Commit message: Added namespace for urdf and now 2 autoserve bots can spawn

File: autoserve_description/urdf/autoserve.xacro (robot description, xacro)
@@ -1,8 +1,10 @@
 <?xml version="1.0" ?>
 <robot name="autoserve" xmlns:xacro="http://www.ros.org/wiki/xacro">
+<xacro:arg name="namespace" default="autoserve"></xacro:arg>
+<xacro:property name="robot_namespace" value="${xacro.arg('namespace')}" />
 <xacro:include filename="$(find autoserve_description)/urdf/materials.xacro" />
 <xacro:include filename="$(find autoserve_description)/urdf/autoserve_gazebo.xacro" />
 <xacro:include filename="$(find autoserve_description)/urdf/autoserve.trans" />
-<link name="base_footprint">
+<link name="${robot_namespace}_base_footprint">
   <!-- <collision>
     <origin xyz="0.0 0.0 0.003" rpy="0 0 0"/>
@@ -12,5 +14,5 @@
   </collision> -->
 </link>
-<link name="base_link">
+<link name="${robot_namespace}_base_link">
   <inertial>
     <origin xyz="0.017764143959187594 -0.00010931568495259127 0.24169621947403908" rpy="0 0 0"/>
@@ -38,11 +40,11 @@
   </collision>
 </link>
-<joint name="footprint2baselink" type="fixed">
-  <parent link="base_footprint"/>
-  <child link="base_link"/>
+<joint name="${robot_namespace}_footprint2baselink" type="fixed">
+  <parent link="${robot_namespace}_base_footprint"/>
+  <child link="${robot_namespace}_base_link"/>
   <origin xyz="0 0 0" rpy="0 0 0"/>
   <axis xyz="0 0 0"/>
 </joint>
-<link name="imu">
+<link name="${robot_namespace}_imu">
   <inertial>
     <origin xyz="-3.552713678800501e-17 -1.7763568394002506e-16 0.0004999999999999727" rpy="0 0 0"/>
@@ -64,5 +66,5 @@
   </collision>
 </link>
-<link name="ydlidar">
+<link name="${robot_namespace}_ydlidar">
   <inertial>
     <origin xyz="-0.030294099570319616 0.03099999999999979 0.037701142222791084" rpy="0 0 0"/>
@@ -84,5 +86,5 @@
   </collision>
 </link>
-<link name="camera_link">
+<link name="${robot_namespace}_camera_link">
   <inertial>
     <origin xyz="0.011951472788559625 0.022747274204167237 -6.086448440437153e-05" rpy="0 0 0"/>
@@ -104,12 +106,12 @@
   </collision>
 </link>
-<link name="camera_link_optical"/>
-<joint name="camera2camera_1" type="fixed">
-  <parent link="camera_link"/>
-  <child link="camera_link_optical"/>
+<link name="${robot_namespace}_camera_link_optical"/>
+<joint name="${robot_namespace}_camera2camera_1" type="fixed">
+  <parent link="${robot_namespace}_camera_link"/>
+  <child link="${robot_namespace}_camera_link_optical"/>
   <origin xyz="0 0 0" rpy="-1.5708 0 -1.5708"/>
   <axis xyz="0 0 0"/>
 </joint>
-<link name="depth_camera_2">
+<link name="${robot_namespace}_depth_camera_2">
   <inertial>
     <origin xyz="0.01195115490287238 0.02274721773464422 -6.09413650859425e-05" rpy="0 0 0"/>
@@ -151,5 +153,5 @@
   </collision>
 </link> -->
-<link name="right_wheel">
+<link name="${robot_namespace}_right_wheel">
   <inertial>
     <origin xyz="1.4446033464149508e-16 -0.015000000000000263 2.0816681711721685e-16" rpy="0 0 0"/>
@@ -171,5 +173,5 @@
   </collision>
 </link>
-<link name="left_wheel">
+<link name="${robot_namespace}_left_wheel">
   <inertial>
     <origin xyz="1.6623077439054263e-16 0.01500000000000018 1.3877787807814457e-16" rpy="0 0 0"/>
@@ -191,5 +193,5 @@
   </collision>
 </link>
-<link name="plate_1">
+<link name="${robot_namespace}_plate_1">
   <inertial>
     <origin xyz="-0.0800003178856868 0.1549999435304768 0.09999999999999992" rpy="0 0 0"/>
@@ -211,5 +213,5 @@
   </collision>
 </link>
-<link name="plate_2">
+<link name="${robot_namespace}_plate_2">
   <inertial>
     <origin xyz="-0.08000031788568687 0.1549999435304768 0.3299999999999999" rpy="0 0 0"/>
@@ -231,18 +233,18 @@
   </collision>
 </link>
-<joint name="base2imu" type="fixed">
+<joint name="${robot_namespace}_base2imu" type="fixed">
   <origin xyz="0.0 0.0 0.203" rpy="0 0 0"/>
-  <parent link="base_link"/>
-  <child link="imu"/>
-</joint>
-<joint name="base2lidar" type="fixed">
+  <parent link="${robot_namespace}_base_link"/>
+  <child link="${robot_namespace}_imu"/>
+</joint>
+<joint name="${robot_namespace}_base2lidar" type="fixed">
   <origin xyz="0.162 0.0 0.25" rpy="0 0 0"/>
-  <parent link="base_link"/>
-  <child link="ydlidar"/>
-</joint>
-<joint name="base2camera_1" type="fixed">
+  <parent link="${robot_namespace}_base_link"/>
+  <child link="${robot_namespace}_ydlidar"/>
+</joint>
+<joint name="${robot_namespace}_base2camera_1" type="fixed">
   <origin xyz="0.2 -0.0 0.1705" rpy="0 0 0"/>
-  <parent link="base_link"/>
-  <child link="camera_link"/>
+  <parent link="${robot_namespace}_base_link"/>
+  <child link="${robot_namespace}_camera_link"/>
 </joint>
 <!-- <joint name="base2camera_2" type="fixed">
@@ -251,33 +253,33 @@
   <child link="depth_camera_2"/>
 </joint> -->
-<joint name="base2camera_2" type="fixed">
+<joint name="${robot_namespace}_base2camera_2" type="fixed">
   <origin xyz="0.105108 -0.0 1.3" rpy="0 0 0"/>
-  <parent link="base_link"/>
-  <child link="depth_camera_2"/>
-</joint>
-<joint name="base2rightw" type="continuous">
+  <parent link="${robot_namespace}_base_link"/>
+  <child link="${robot_namespace}_depth_camera_2"/>
+</joint>
+<joint name="${robot_namespace}_base2rightw" type="continuous">
   <origin xyz="0.0 -0.1659 0.05" rpy="0 0 0"/>
-  <parent link="base_link"/>
-  <child link="right_wheel"/>
+  <parent link="${robot_namespace}_base_link"/>
+  <child link="${robot_namespace}_right_wheel"/>
   <axis xyz="-0.0 1.0 0.0"/>
 </joint>
-<joint name="base2leftw" type="continuous">
+<joint name="${robot_namespace}_base2leftw" type="continuous">
   <origin xyz="0.0 0.1659 0.05" rpy="0 0 0"/>
-  <parent link="base_link"/>
-  <child link="left_wheel"/>
+  <parent link="${robot_namespace}_base_link"/>
+  <child link="${robot_namespace}_left_wheel"/>
   <axis xyz="0.0 1.0 0.0"/>
 </joint>
 <!-- prismatic -->
-<joint name="base2plate_1" type="prismatic">
+<joint name="${robot_namespace}_base2plate_1" type="prismatic">
   <origin xyz="0.0 -0.0 0.303" rpy="0 0 0"/>
-  <parent link="base_link"/>
-  <child link="plate_1"/>
+  <parent link="${robot_namespace}_base_link"/>
+  <child link="${robot_namespace}_plate_1"/>
   <axis xyz="1.0 -0.0 -0.0"/>
   <limit upper="0.08" lower="-0.08" effort="100" velocity="100"/>
 </joint>
-<joint name="base2plate_2" type="prismatic">
+<joint name="${robot_namespace}_base2plate_2" type="prismatic">
   <origin xyz="0.0 -0.0 0.533" rpy="0 0 0"/>
-  <parent link="base_link"/>
-  <child link="plate_2"/>
+  <parent link="${robot_namespace}_base_link"/>
+  <child link="${robot_namespace}_plate_2"/>
   <axis xyz="1.0 -0.0 -0.0"/>
   <limit upper="0.08" lower="-0.08" effort="100" velocity="100"/>

File: autoserve_description/urdf/autoserve_gazebo.xacro (robot description, xacro)
@@ -8,16 +8,16 @@
 <xacro:property name="plate" value="Gazebo/Green" />
   <!-- Wheels -->
-  <gazebo reference="left_wheel">
+  <gazebo reference="${robot_namespace}_left_wheel">
     <material>${wheels}</material>
-    <mu1>1000.0</mu1>
-    <mu2>1000.0</mu2>
+    <mu1>0.1</mu1>
+    <mu2>0.1</mu2>
     <maxContacts>1</maxContacts>
     <selfCollide>true</selfCollide>
     <gravity>true</gravity>
   </gazebo>
-  <gazebo reference="right_wheel">
+  <gazebo reference="${robot_namespace}_right_wheel">
     <material>${wheels}</material>
-    <mu1>1000.0</mu1>
-    <mu2>1000.0</mu2>
+    <mu1>0.1</mu1>
+    <mu2>0.1</mu2>
     <maxContacts>1</maxContacts>
     <selfCollide>true</selfCollide>
@@ -25,5 +25,5 @@
   </gazebo>
   <!-- Caster Wheels -->
-  <gazebo reference="base_link">
+  <gazebo reference="${robot_namespace}_base_link">
     <material>${base_link}</material>
     <mu1>0.1</mu1>
@@ -33,35 +33,35 @@
     <gravity>true</gravity>
   </gazebo>
-  <gazebo reference="base_footprint">
-    <mu1>0.1</mu1>
-    <mu2>0.1</mu2>
-    <maxContacts>1</maxContacts>
-  </gazebo>
-  <gazebo reference="depth_camera_1">
+  <gazebo reference="${robot_namespace}_base_footprint">
+    <mu1>0.1</mu1>
+    <mu2>0.1</mu2>
+    <maxContacts>1</maxContacts>
+  </gazebo>
+  <gazebo reference="${robot_namespace}_depth_camera_1">
     <material>${depth_cam}</material>
     <mu1>0.1</mu1>
     <mu2>0.1</mu2>
   </gazebo>
-  <gazebo reference="depth_camera_2">
+  <gazebo reference="${robot_namespace}_depth_camera_2">
     <material>${depth_cam}</material>
     <mu1>0.1</mu1>
     <mu2>0.1</mu2>
   </gazebo>
-  <gazebo reference="ydlidar">
+  <gazebo reference="${robot_namespace}_ydlidar">
     <material>${lidar}</material>
     <mu1>0.1</mu1>
     <mu2>0.1</mu2>
   </gazebo>
-  <gazebo reference="imu">
+  <gazebo reference="${robot_namespace}_imu">
     <material>${imu}</material>
     <mu1>0.1</mu1>
     <mu2>0.1</mu2>
   </gazebo>
-  <gazebo reference="plate_1">
+  <gazebo reference="${robot_namespace}_plate_1">
     <material>${plate}</material>
     <mu1>0.1</mu1>
     <mu2>0.1</mu2>
   </gazebo>
-  <gazebo reference="plate_2">
+  <gazebo reference="${robot_namespace}_plate_2">
     <material>${plate}</material>
     <mu1>0.1</mu1>
@@ -75,5 +75,5 @@
     </plugin>
   </gazebo> -->
-  <gazebo>
+  <!-- <gazebo>
     <plugin name="diff_drive_control" filename="libgazebo_ros_diff_drive.so">
       <update_rate>50</update_rate>
@@ -90,21 +90,34 @@
       <robot_base_frame>base_footprint</robot_base_frame>
     </plugin>
-  </gazebo>
-  <gazebo reference="imu">
-    <gravity>true</gravity>
-    <sensor name="imu" type="imu">
+  </gazebo> -->
+  <gazebo>
+    <plugin name="${robot_namespace}_object_controller" filename="libgazebo_ros_planar_move.so">
+        <ros>
+          <!-- <namespace>${robot_namespace}</namespace> -->
+          <remapping>cmd_vel:=${robot_namespace}_cmd_vel</remapping>
+          <remapping>odom:=${robot_namespace}_odom</remapping>
+      </ros>
+      <odometry_frame>odom</odometry_frame>
+      <update_rate>20.0</update_rate>
+      <publish_rate>20.0</publish_rate>
+      <robot_base_frame>${robot_namespace}_base_footprint</robot_base_frame>
+    </plugin>
+  </gazebo>
+  <gazebo reference="${robot_namespace}_imu">
+    <gravity>true</gravity>
+    <sensor name="${robot_namespace}_imu" type="imu">
       <always_on>true</always_on>
       <update_rate>30</update_rate>
       <visualize>true</visualize>
-      <plugin name="my_imu_plugin" filename="libgazebo_ros_imu_sensor.so">
+      <plugin name="${robot_namespace}_my_imu_plugin" filename="libgazebo_ros_imu_sensor.so">
         <ros>
-          <remapping>~/out:=imu</remapping>
+          <remapping>~/out:=${robot_namespace}_imu</remapping>
         </ros>
-        <frame_name>imu</frame_name>
-      </plugin>
-    </sensor>
-  </gazebo>
-  <gazebo reference="ydlidar">
-    <sensor type="ray" name="head_hokuyo_sensor">
+        <frame_name>${robot_namespace}_imu</frame_name>
+      </plugin>
+    </sensor>
+  </gazebo>
+  <gazebo reference="${robot_namespace}_ydlidar">
+    <sensor type="ray" name="${robot_namespace}_head_hokuyo_sensor">
       <pose>0 0 0 0 0 0</pose>
       <visualize>false</visualize>
@@ -130,20 +143,20 @@
         </noise>
       </ray>
-      <plugin name="my_ray_sensor_plugin" filename="libgazebo_ros_ray_sensor.so">
+      <plugin name="${robot_namespace}_my_ray_sensor_plugin" filename="libgazebo_ros_ray_sensor.so">
         <ros>
-          <remapping>~/out:=scan</remapping>
+          <remapping>~/out:=${robot_namespace}_scan</remapping>
         </ros>
         <output_type>sensor_msgs/LaserScan</output_type>
         <min_intensity>100.0</min_intensity>
-        <frame_name>ydlidar</frame_name>
-      </plugin>
-    </sensor>
-  </gazebo>
-  <gazebo reference="camera_link">
-    <sensor name="camera" type="depth">
+        <frame_name>${robot_namespace}_ydlidar</frame_name>
+      </plugin>
+    </sensor>
+  </gazebo>
+  <gazebo reference="${robot_namespace}_camera_link">
+    <sensor name="${robot_namespace}_camera" type="depth">
       <pose> 0 0 0 0 0 0</pose>
       <visualize>true</visualize>
       <update_rate>60.0</update_rate>
-      <camera name="camera_link">
+      <camera name="${robot_namespace}_camera_link">
         <horizontal_fov>1.047198</horizontal_fov>
         <image>
@@ -157,9 +170,9 @@
         </clip>
       </camera>
-      <plugin name="depth_camera_controller_1" filename="libgazebo_ros_camera.so">
+      <plugin name="${robot_namespace}_depth_camera_controller_1" filename="libgazebo_ros_camera.so">
         <baseline>0.2</baseline>
         <alwaysOn>true</alwaysOn>
         <updateRate>0.0</updateRate>
-        <frame_name>camera_link_optical</frame_name>
+        <frame_name>${robot_namespace}_camera_link_optical</frame_name>
         <pointCloudCutoff>0.1</pointCloudCutoff>
         <pointCloudCutoffMax>50.0</pointCloudCutoffMax>
@@ -177,10 +190,10 @@
     </sensor>
   </gazebo>
-  <gazebo reference="depth_camera_2">
-    <sensor name="camera_2" type="depth">
+  <gazebo reference="${robot_namespace}_depth_camera_2">
+    <sensor name="${robot_namespace}_camera_2" type="depth">
       <pose> 0 0 0 0 0 0</pose>
       <visualize>true</visualize>
       <update_rate>60.0</update_rate>
-      <camera name="depth_camera_2">
+      <camera name="${robot_namespace}_depth_camera_2">
         <horizontal_fov>1.047198</horizontal_fov>
         <image>
@@ -194,9 +207,9 @@
         </clip>
       </camera>
-      <plugin name="depth_camera_controller_2" filename="libgazebo_ros_camera.so">
+      <plugin name="${robot_namespace}_depth_camera_controller_2" filename="libgazebo_ros_camera.so">
         <baseline>0.2</baseline>
         <alwaysOn>true</alwaysOn>
         <updateRate>0.0</updateRate>
-        <frame_name>depth_camera_2</frame_name>
+        <frame_name>${robot_namespace}_depth_camera_2</frame_name>
         <pointCloudCutoff>0.1</pointCloudCutoff>
         <pointCloudCutoffMax>10.0</pointCloudCutoffMax>

File: autoserve_description/urdf/autoserve_ros2_control.xacro (robot description, xacro)
@@ -5,5 +5,5 @@
             <plugin>gazebo_ros2_control/GazeboSystem</plugin>
         </hardware>
-        <joint name="base2plate_1">
+        <joint name="${robot_namespace}_base2plate_1">
             <command_interface name="position">
               <param name="min">-0.8</param>
@@ -12,5 +12,5 @@
             <state_interface name="position" />
         </joint>
-        <joint name="base2plate_2">
+        <joint name="${robot_namespace}_base2plate_2">
             <command_interface name="position">
               <param name="min">-0.8</param>

Commit message: Refactor URDF and launch files: update mass values, rename camera links, adjust friction parameters for wheels, and enable verbose mode in Gazebo launch configuration.

File: autoserve_description/urdf/autoserve.xacro (robot description, xacro)
@@ -4,4 +4,5 @@
 <xacro:include filename="$(find autoserve_description)/urdf/autoserve_gazebo.xacro" />
 <xacro:include filename="$(find autoserve_description)/urdf/autoserve.trans" />
+<!-- <xacro:include filename="$(find autoserve_description)/urdf/autoserve_ros2_control.xacro" /> -->
 <link name="base_footprint">
   <!-- <collision>
@@ -15,5 +16,5 @@
   <inertial>
     <origin xyz="0.017764143959187594 -0.00010931568495259127 0.24169621947403908" rpy="0 0 0"/>
-    <mass value="10.036859574001216"/>
+    <mass value="30.036859574001216"/>
     <inertia ixx="0.822232" iyy="0.810255" izz="0.334887" ixy="-1.8e-05" iyz="0.000454" ixz="-0.000983"/>
   </inertial>
@@ -84,5 +85,5 @@
   </collision>
 </link>
-<link name="camera_link">
+<link name="depth_camera_1">
   <inertial>
     <origin xyz="0.011951472788559625 0.022747274204167237 -6.086448440437153e-05" rpy="0 0 0"/>
@@ -104,8 +105,8 @@
   </collision>
 </link>
-<link name="camera_link_optical"/>
-<joint name="camera2camera_1" type="fixed">
-  <parent link="camera_link"/>
-  <child link="camera_link_optical"/>
+<link name="camera_link_1_optical"/>
+<joint name="dcamera2camera_1" type="fixed">
+  <parent link="depth_camera_1"/>
+  <child link="camera_link_1_optical"/>
   <origin xyz="0 0 0" rpy="-1.5708 0 -1.5708"/>
   <axis xyz="0 0 0"/>
@@ -265,5 +266,5 @@
   <origin xyz="0.2 -0.0 0.1705" rpy="0 0 0"/>
   <parent link="base_link"/>
-  <child link="camera_link"/>
+  <child link="depth_camera_1"/>
 </joint>
 <joint name="base2camera_2" type="fixed">

File: autoserve_description/urdf/autoserve_gazebo.xacro (robot description, xacro)
@@ -10,27 +10,27 @@
   <gazebo reference="left_wheel">
     <material>${wheels}</material>
-    <mu1>1000.0</mu1>
-    <mu2>1000.0</mu2>
+    <mu1>100.0</mu1>
+    <mu2>100.0</mu2>
+    <maxContacts>10</maxContacts>
+    <selfCollide>true</selfCollide>
+    <gravity>true</gravity>
+  </gazebo>
+  <gazebo reference="right_wheel">
+    <material>${wheels}</material>
+    <mu1>100.0</mu1>
+    <mu2>100.0</mu2>
+    <maxContacts>10</maxContacts>
+    <selfCollide>true</selfCollide>
+    <gravity>true</gravity>
+  </gazebo>
+  <!-- Caster Wheels -->
+  <gazebo reference="base_link">
+    <material>${base_link}</material>
+    <mu1>0.25</mu1>
+    <mu2>0.25</mu2>
     <maxContacts>1</maxContacts>
     <selfCollide>true</selfCollide>
     <gravity>true</gravity>
   </gazebo>
-  <gazebo reference="right_wheel">
-    <material>${wheels}</material>
-    <mu1>1000.0</mu1>
-    <mu2>1000.0</mu2>
-    <maxContacts>1</maxContacts>
-    <selfCollide>true</selfCollide>
-    <gravity>true</gravity>
-  </gazebo>
-  <!-- Caster Wheels -->
-  <gazebo reference="base_link">
-    <material>${base_link}</material>
-    <mu1>0.1</mu1>
-    <mu2>0.1</mu2>
-    <maxContacts>1</maxContacts>
-    <selfCollide>true</selfCollide>
-    <gravity>true</gravity>
-  </gazebo>
   <gazebo reference="base_footprint">
     <mu1>0.1</mu1>
@@ -69,5 +69,5 @@
   </gazebo>
   <!-- <gazebo>
-    <plugin filename="libgazebo_ros2_control.so" name="gazebo_ros2_control">
+    <plugin filename="libgazebo_ros2_control.so" name="gazebo_ros2_control_autoserve">
       <robot_param>robot_description</robot_param>
       <robot_param_node>robot_state_publisher</robot_param_node>
@@ -77,7 +77,4 @@
   <gazebo>
     <plugin name="diff_drive_control" filename="libgazebo_ros_diff_drive.so">
-      <!-- <ros>
-        <remapping>/cmd_vel:=/cmd_vel_new</remapping>
-      </ros> -->
       <update_rate>20</update_rate>
       <left_joint>base2leftw</left_joint>
@@ -288,10 +285,10 @@
     </sensor>
   </gazebo>
-  <gazebo reference="camera_link">
+  <gazebo reference="depth_camera_1">
     <sensor name="camera" type="depth">
       <pose> 0 0 0 0 0 0</pose>
       <visualize>true</visualize>
       <update_rate>10.0</update_rate>
-      <camera name="camera_link">
+      <camera name="depth_camera_2">
         <horizontal_fov>1.57</horizontal_fov>
         <image>
@@ -309,5 +306,5 @@
         <alwaysOn>true</alwaysOn>
         <updateRate>0.0</updateRate>
-        <frame_name>camera_link_optical</frame_name>
+        <frame_name>camera_link_1_optical</frame_name>
         <pointCloudCutoff>0.1</pointCloudCutoff>
         <pointCloudCutoffMax>5.0</pointCloudCutoffMax>

File: autoserve_description/urdf/autoserve_ros2_control.xacro (robot description, xacro)
@@ -5,5 +5,5 @@
             <plugin>gazebo_ros2_control/GazeboSystem</plugin>
         </hardware>
-        <joint name="base2plate_1">
+        <!-- <joint name="base2plate_1">
             <command_interface name="position">
               <param name="min">-0.8</param>
@@ -18,6 +18,6 @@
             </command_interface>
             <state_interface name="position" />
-        </joint>
-        <!-- <joint name="base2leftw">
+        </joint> -->
+        <joint name="base2leftw">
             <command_interface name="velocity">
               <param name="min">-10</param>
@@ -34,5 +34,5 @@
             <state_interface name="position" />
             <state_interface name="velocity" />
-        </joint> -->
+        </joint>
     </ros2_control>
 </robot>
