Commit message: Refactor URDF and Gazebo launch files: update mass values for base link, adjust friction coefficients for wheels, and clean up commented gazebo plugin sections.

File: autoserve_description/urdf/autoserve.xacro (robot description, xacro)
@@ -6,36 +6,36 @@
 <!-- <xacro:include filename="$(find autoserve_description)/urdf/autoserve_ros2_control.xacro" /> -->
 <link name="base_footprint">
+  <collision>
+    <origin xyz="0.0 0.0 0.003" rpy="0 0 0"/>
+    <geometry>
+      <box size="0.4 0.20 0.005" />
+    </geometry>
+  </collision>
+</link>
+<link name="base_link">
+  <inertial>
+    <origin xyz="0.017764143959187594 -0.00010931568495259127 0.24169621947403908" rpy="0 0 0"/>
+    <mass value="2.036859574001216"/>
+    <inertia ixx="0.822232" iyy="0.810255" izz="0.334887" ixy="-1.8e-05" iyz="0.000454" ixz="-0.000983"/>
+  </inertial>
+  <visual>
+    <origin xyz="0 0 0" rpy="0 0 0"/>
+    <geometry>
+      <mesh filename="package://autoserve_description/meshes/base_link.stl" scale="0.001 0.001 0.001"/>
+    </geometry>
+    <material name="plastic_translucent_matte_green"/>
+  </visual>
+  <collision>
+    <origin xyz="0 0 0" rpy="0 0 0"/>
+    <geometry>
+      <mesh filename="package://autoserve_description/meshes/base_link.stl" scale="0.001 0.001 0.001"/>
+    </geometry>
+  </collision>
   <!-- <collision>
     <origin xyz="0.0 0.0 0.003" rpy="0 0 0"/>
     <geometry>
-      <box size="0.4 0.20 0.005" />
+      <box size="0.45 0.20 0.005" />
     </geometry>
   </collision> -->
-</link>
-<link name="base_link">
-  <inertial>
-    <origin xyz="0.017764143959187594 -0.00010931568495259127 0.24169621947403908" rpy="0 0 0"/>
-    <mass value="30.036859574001216"/>
-    <inertia ixx="0.822232" iyy="0.810255" izz="0.334887" ixy="-1.8e-05" iyz="0.000454" ixz="-0.000983"/>
-  </inertial>
-  <visual>
-    <origin xyz="0 0 0" rpy="0 0 0"/>
-    <geometry>
-      <mesh filename="package://autoserve_description/meshes/base_link.stl" scale="0.001 0.001 0.001"/>
-    </geometry>
-    <material name="plastic_translucent_matte_green"/>
-  </visual>
-  <collision>
-    <origin xyz="0 0 0" rpy="0 0 0"/>
-    <geometry>
-      <mesh filename="package://autoserve_description/meshes/base_link.stl" scale="0.001 0.001 0.001"/>
-    </geometry>
-  </collision>
-  <collision>
-    <origin xyz="0.0 0.0 0.003" rpy="0 0 0"/>
-    <geometry>
-      <box size="0.45 0.20 0.005" />
-    </geometry>
-  </collision>
 </link>
 <joint name="footprint2baselink" type="fixed">

File: autoserve_description/urdf/autoserve_gazebo.xacro (robot description, xacro)
@@ -10,6 +10,6 @@
   <gazebo reference="left_wheel">
     <material>${wheels}</material>
-    <mu1>100.0</mu1>
-    <mu2>100.0</mu2>
+    <mu1>10.0</mu1>
+    <mu2>10.0</mu2>
     <maxContacts>10</maxContacts>
     <selfCollide>true</selfCollide>
@@ -18,6 +18,6 @@
   <gazebo reference="right_wheel">
     <material>${wheels}</material>
-    <mu1>100.0</mu1>
-    <mu2>100.0</mu2>
+    <mu1>10.0</mu1>
+    <mu2>10.0</mu2>
     <maxContacts>10</maxContacts>
     <selfCollide>true</selfCollide>
@@ -75,5 +75,5 @@
     </plugin>
   </gazebo> -->
-  <gazebo>
+  <!-- <gazebo>
     <plugin name="diff_drive_control" filename="libgazebo_ros_diff_drive.so">
       <update_rate>20</update_rate>
@@ -89,5 +89,5 @@
       <robot_base_frame>base_footprint</robot_base_frame>
     </plugin>
-  </gazebo>
+  </gazebo> -->
   <gazebo reference="imu">
     <gravity>true</gravity>

Commit message: stvl clearing

File: autoserve_description/urdf/autoserve.xacro (robot description, xacro)
@@ -263,5 +263,5 @@
 </joint>
 <joint name="base2camera_1" type="fixed">
-  <origin xyz="0.2 -0.0 0.1705" rpy="0 0 0"/>
+  <origin xyz="0.2 -0.0 0.1705" rpy="0 -0.5 0"/>
   <parent link="base_link"/>
   <child link="camera_link"/>

File: autoserve_description/urdf/autoserve_gazebo.xacro (robot description, xacro)
@@ -292,5 +292,5 @@
       <pose> 0 0 0 0 0 0</pose>
       <visualize>true</visualize>
-      <update_rate>10.0</update_rate>
+      <update_rate>30.0</update_rate>
       <camera name="camera_link">
         <horizontal_fov>1.57</horizontal_fov>
